File: power-amp.sch (KiCad schematic (older format))
At the start: 45 parts, among them J1 JST_XH_3, J2 JST_XH_2, J3 JST_XH_2, J4 Conn_01x02_Male, J6 JST_XH_3, U1 NE5532, U2 LM3886, U3 LM3886

Commit message: fixed resistor values
Parts:
- R1, R10, R11, R12, R4, R5, R6, R7, R8, R9: symbol custom:R_Small -> power-amp-rescue:R_Small-custom
- R13, R14, R2, R3: value 1K 1W -> 2K 1W; symbol custom:R_Small -> power-amp-rescue:R_Small-custom
Other:
- note removed: "68u: A767MU107M1HLAE027"
Changed lines of the file:
@@
 EESchema Schematic File Version 4
 LIBS:power-amp-cache
-EELAYER 29 0
+EELAYER 26 0
 EELAYER END
 $Descr A4 11693 8268
@@
 	4400 2875 4400 3150
 $Comp
-L custom:R_Small R7
+L power-amp-rescue:R_Small-custom R7
 U 1 1 5CDC3A8A
 P 4400 3275
@@
 $EndComp
 $Comp
-L custom:R_Small R5
+L power-amp-rescue:R_Small-custom R5
 U 1 1 5CDC4124
 P 3925 2675
@@
 	4025 2675 4500 2675
 $Comp
-L custom:R_Small R9
+L power-amp-rescue:R_Small-custom R9
 U 1 1 5CDDD6F2
 P 4950 3150
@@
 	5150 3150 5150 2775
 $Comp
-L custom:R_Small R11
+L power-amp-rescue:R_Small-custom R11
 U 1 1 5CDE1752
 P 5350 2775
@@
 	4400 4625 4400 4900
 $Comp
-L custom:R_Small R8
+L power-amp-rescue:R_Small-custom R8
 U 1 1 5CDE2496
 P 4400 5025
@@
 $EndComp
 $Comp
-L custom:R_Small R6
+L power-amp-rescue:R_Small-custom R6
 U 1 1 5CDE24A0
 P 3925 4425
@@
 	4025 4425 4500 4425
 $Comp
-L custom:R_Small R10
+L power-amp-rescue:R_Small-custom R10
 U 1 1 5CDE24AB
 P 4950 4900
@@
 	3800 4425 3825 4425
 $Comp
-L custom:R_Small R4
+L power-amp-rescue:R_Small-custom R4
 U 1 1 5CDECF2B
 P 3525 3750
@@
 $EndComp
 $Comp
-L custom:R_Small R1
+L power-amp-rescue:R_Small-custom R1
 U 1 1 5CE5DCAE
 P 1475 3600
@@
 Wire Wire Line
 	7950 1025 7950 1075
-Text Notes 8950 875  0    50   ~ 0
-68u: A767MU107M1HLAE027
-$Comp
-L custom:R_Small R12
+$Comp
+L power-amp-rescue:R_Small-custom R12
 U 1 1 5CF69493
 P 5350 4525
@@
 $EndComp
 $Comp
-L custom:R_Small R2
+L power-amp-rescue:R_Small-custom R2
 U 1 1 5CE64E43
 P 1950 1025
 F 0 "R2" H 2050 1000 50  0000 C CNN
-F 1 "1K 1W" H 2125 1075 50  0000 C CNN
+F 1 "2K 1W" H 2125 1075 50  0000 C CNN
 F 2 "Resistor_SMD:R_1206_3216Metric" H 1950 1025 50  0001 C CNN
 F 3 "" H 1950 1025 50  0001 C CNN
@@
 	2025 900  2025 925
 $Comp
-L custom:R_Small R13
+L power-amp-rescue:R_Small-custom R13
 U 1 1 5CE83E7E
 P 3300 1250
 F 0 "R13" H 3400 1225 50  0000 C CNN
-F 1 "1K 1W" H 3475 1300 50  0000 C CNN
+F 1 "2K 1W" H 3475 1300 50  0000 C CNN
 F 2 "Resistor_SMD:R_1206_3216Metric" H 3300 1250 50  0001 C CNN
 F 3 "" H 3300 1250 50  0001 C CNN
@@
 $EndComp
 $Comp
-L custom:R_Small R3
+L power-amp-rescue:R_Small-custom R3
 U 1 1 5CE844D1
 P 2025 1025
 F 0 "R3" H 2125 1000 50  0000 C CNN
-F 1 "1K 1W" H 2200 1075 50  0000 C CNN
+F 1 "2K 1W" H 2200 1075 50  0000 C CNN
 F 2 "Resistor_SMD:R_1206_3216Metric" H 2025 1025 50  0001 C CNN
 F 3 "" H 2025 1025 50  0001 C CNN
@@
 $EndComp
 $Comp
-L custom:R_Small R14
+L power-amp-rescue:R_Small-custom R14
 U 1 1 5CE84735
 P 3400 1250
 F 0 "R14" H 3500 1225 50  0000 C CNN
-F 1 "1K 1W" H 3575 1300 50  0000 C CNN
+F 1 "2K 1W" H 3575 1300 50  0000 C CNN
 F 2 "Resistor_SMD:R_1206_3216Metric" H 3400 1250 50  0001 C CNN
 F 3 "" H 3400 1250 50  0001 C CNN
